File: kicad/rev.2.0/DiLight_2.0.kicad_sch (KiCad schematic)
At the start: 21 parts, among them J1 12V IN, J2 LED strip, J3 Sensor, J4 Touch, J5 ST Link V3, Q1 AP4435C, Q2 AO3400A, U1 AMS1117-3.3, U2 STM32G031G8Ux

Commit message: BOM status changed for some components. iBOM regenerated
Parts:
- H1, H2: now left out of the parts list
Changed lines of the file:
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@@
   )
   (symbol (lib_id "Mechanical:MountingHole") (at 113.665 126.365 0) (unit 1)
-    (in_bom yes) (on_board yes) (fields_autoplaced)
+    (in_bom no) (on_board yes) (fields_autoplaced)
     (property "Reference" "H1" (id 0) (at 116.205 125.5303 0)
       (effects (font (size 1.27 1.27)) (justify left))
@@
   )
   (symbol (lib_id "Mechanical:MountingHole") (at 113.665 131.445 0) (unit 1)
-    (in_bom yes) (on_board yes) (fields_autoplaced)
+    (in_bom no) (on_board yes) (fields_autoplaced)
     (property "Reference" "H2" (id 0) (at 116.205 130.6103 0)
       (effects (font (size 1.27 1.27)) (justify left))
